File: Hardware/3-pin digital LED corner PCB.kicad_pcb (KiCad board)
At the start: 2 copper layers, 20.5 x 20.5 mm, 15 parts, among them J1 Conn_01x01_Male, J2 Conn_01x01_Male, J3 Conn_01x01_Male, J4 Conn_01x01_Male, J5 Conn_01x01_Male, J6 Conn_01x01_Male

Commit message: Update 3-pin digital LED corner PCB.kicad_pcb
Parts:
- added G***: LOGO, LOGO, B.Cu at (144.8, 119.8)
Other:
- board text added: "3 Pin Dig. LED Corner V1"

Commit message: update to 2 and 3 pin corner PCB
Parts:
- added J10: Conn_01x01_Male, TestPoint:TestPoint_Pad_2.0x2.0mm, B.Cu at (146.4, 105.3)
- added J10: Conn_01x01_Male, TestPoint:TestPoint_Pad_2.0x2.0mm, B.Cu at (147.9, 105.3)
- added J10: Conn_01x01_Male, TestPoint:TestPoint_Pad_2.0x2.0mm, B.Cu at (146.4, 107.3)
- added J10: Conn_01x01_Male, TestPoint:TestPoint_Pad_2.0x2.0mm, B.Cu at (147.9, 107.3)
- added J7: Conn_01x01_Male, TestPoint:TestPoint_Pad_2.0x2.0mm, B.Cu at (157.2, 121.6)
- added J7: Conn_01x01_Male, TestPoint:TestPoint_Pad_2.0x2.0mm, B.Cu at (159.2, 123.5)
- added J7: Conn_01x01_Male, TestPoint:TestPoint_Pad_2.0x2.0mm, B.Cu at (157.2, 123.5)
- added J7: Conn_01x01_Male, TestPoint:TestPoint_Pad_2.0x2.0mm, B.Cu at (159.2, 121.6)
- added J8: Conn_01x01_Male, TestPoint:TestPoint_Pad_2.0x2.0mm, B.Cu at (157.2, 116.2)
- added J8: Conn_01x01_Male, TestPoint:TestPoint_Pad_2.0x2.0mm, B.Cu at (159.2, 118.1)
- added J8: Conn_01x01_Male, TestPoint:TestPoint_Pad_2.0x2.0mm, B.Cu at (157.2, 118.1)
- added J8: Conn_01x01_Male, TestPoint:TestPoint_Pad_2.0x2.0mm, B.Cu at (159.2, 116.2)
- added J9: Conn_01x01_Male, TestPoint:TestPoint_Pad_2.0x2.0mm, B.Cu at (143.1, 107.3)
- added J9: Conn_01x01_Male, TestPoint:TestPoint_Pad_2.0x2.0mm, B.Cu at (141.3, 105.3)
- added J9: Conn_01x01_Male, TestPoint:TestPoint_Pad_2.0x2.0mm, B.Cu at (141.3, 107.3)
- added J9: Conn_01x01_Male, TestPoint:TestPoint_Pad_2.0x2.0mm, B.Cu at (143.1, 105.3)
Routing:
- added copper zone on B.Cu, net /2pin1
- added copper zone on B.Cu, net /2pin2
Other:
- board text added: "1"
- board text added: "2"
- board text added: "2/3 Pin LED Corner V2"
- board text added: "V+"
- board text added: "V-"
- board text removed: "3 Pin Dig. LED Corner V1"
