File: Hardware/3-pin digital LED corner PCB.kicad_sch (KiCad schematic)
At the start: 9 parts, among them J1 Conn_01x01_Male, J2 Conn_01x01_Male, J3 Conn_01x01_Male, J4 Conn_01x01_Male, J5 Conn_01x01_Male, J6 Conn_01x01_Male

Commit message: update to 2 and 3 pin corner PCB
Parts:
- added J10, J7, J8, J9: Conn_01x01_Male, TestPoint:TestPoint_Pad_2.0x2.0mm, symbol Connector:Conn_01x01_Male
Connections:
- new net 2pin1: J7.1 (Pin_1), J9.1 (Pin_1)
- new net 2pin2: J10.1 (Pin_1), J8.1 (Pin_1)
Changed lines of the file:
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@@
+    (stroke (width 0) (type default) (color 0 0 0 0))
+  )
+  (wire (pts (xy 163.83 120.65) (xy 172.72 120.65))
     (stroke (width 0) (type default) (color 0 0 0 0))
   )
@@
     (stroke (width 0) (type default) (color 0 0 0 0))
   )
+  (wire (pts (xy 163.83 118.11) (xy 172.72 118.11))
+    (stroke (width 0) (type default) (color 0 0 0 0))
+  )
   (wire (pts (xy 167.64 90.17) (xy 171.45 90.17))
     (stroke (width 0) (type default) (color 0 0 0 0))
@@
   (wire (pts (xy 125.73 88.9) (xy 125.73 87.63))
     (stroke (width 0) (type default) (color 0 0 0 0))
+  )
+  (label "2pin2" (at 166.37 120.65 0)
+    (effects (font (size 1.27 1.27)) (justify left bottom))
+  )
+  (label "2pin1" (at 166.37 118.11 0)
+    (effects (font (size 1.27 1.27)) (justify left bottom))
   )
   (symbol (lib_id "LED:WS2812B") (at 146.05 92.71 0) (unit 1)
@@
     (pin "1")
   )
+  (symbol (lib_id "Connector:Conn_01x01_Male") (at 158.75 118.11 0) (unit 1)
+    (in_bom yes) (on_board yes)
+    (property "Reference" "J7" (id 0) (at 138.43 118.11 0))
+    (property "Value" "Conn_01x01_Male" (id 1) (at 148.59 118.11 0))
+    (property "Footprint" "TestPoint:TestPoint_Pad_2.0x2.0mm" (id 2) (at 158.75 118.11 0)
+      (effects (font (size 1.27 1.27)) hide)
+    )
+    (property "Datasheet" "~" (id 3) (at 158.75 118.11 0)
+      (effects (font (size 1.27 1.27)) hide)
+    )
+    (pin "1")
+  )
+  (symbol (lib_id "Connector:Conn_01x01_Male") (at 158.75 120.65 0) (unit 1)
+    (in_bom yes) (on_board yes)
+    (property "Reference" "J8" (id 0) (at 138.43 120.65 0))
+    (property "Value" "Conn_01x01_Male" (id 1) (at 148.59 120.65 0))
+    (property "Footprint" "TestPoint:TestPoint_Pad_2.0x2.0mm" (id 2) (at 158.75 120.65 0)
+      (effects (font (size 1.27 1.27)) hide)
+    )
+    (property "Datasheet" "~" (id 3) (at 158.75 120.65 0)
+      (effects (font (size 1.27 1.27)) hide)
+    )
+    (pin "1")
+  )
   (symbol (lib_id "Connector:Conn_01x01_Male") (at 115.57 92.71 0) (unit 1)
     (in_bom yes) (on_board yes)
@@
     (pin "1")
   )
+  (symbol (lib_id "Connector:Conn_01x01_Male") (at 177.8 118.11 180) (unit 1)
+    (in_bom yes) (on_board yes)
+    (property "Reference" "J9" (id 0) (at 198.12 118.11 0))
+    (property "Value" "Conn_01x01_Male" (id 1) (at 187.96 118.11 0))
+    (property "Footprint" "TestPoint:TestPoint_Pad_2.0x2.0mm" (id 2) (at 177.8 118.11 0)
+      (effects (font (size 1.27 1.27)) hide)
+    )
+    (property "Datasheet" "~" (id 3) (at 177.8 118.11 0)
+      (effects (font (size 1.27 1.27)) hide)
+    )
+    (pin "1")
+  )
   (symbol (lib_id "Device:C") (at 130.81 92.71 0) (unit 1)
     (in_bom yes) (on_board yes) (fields_autoplaced)
@@
     (pin "1")
   )
+  (symbol (lib_id "Connector:Conn_01x01_Male") (at 177.8 120.65 180) (unit 1)
+    (in_bom yes) (on_board yes)
+    (property "Reference" "J10" (id 0) (at 198.12 120.65 0))
+    (property "Value" "Conn_01x01_Male" (id 1) (at 187.96 120.65 0))
+    (property "Footprint" "TestPoint:TestPoint_Pad_2.0x2.0mm" (id 2) (at 177.8 120.65 0)
+      (effects (font (size 1.27 1.27)) hide)
+    )
+    (property "Datasheet" "~" (id 3) (at 177.8 120.65 0)
+      (effects (font (size 1.27 1.27)) hide)
+    )
+    (pin "1")
+  )
   (sheet_instances
     (path "/" (page "1"))
@@
       (reference "J6") (unit 1) (value "Conn_01x01_Male") (footprint "TestPoint:TestPoint_Pad_2.0x2.0mm")
     )
+    (path "/760f49b2-3b1f-4100-9d74-d73c84ac5cd9"
+      (reference "J7") (unit 1) (value "Conn_01x01_Male") (footprint "TestPoint:TestPoint_Pad_2.0x2.0mm")
+    )
+    (path "/770267bd-6b08-4ce9-9859-255364603a92"
+      (reference "J8") (unit 1) (value "Conn_01x01_Male") (footprint "TestPoint:TestPoint_Pad_2.0x2.0mm")
+    )
+    (path "/9aba9eaa-06af-4d38-b822-b427891cc96f"
+      (reference "J9") (unit 1) (value "Conn_01x01_Male") (footprint "TestPoint:TestPoint_Pad_2.0x2.0mm")
+    )
+    (path "/ee7c5229-8122-44df-afad-d951332531ee"
+      (reference "J10") (unit 1) (value "Conn_01x01_Male") (footprint "TestPoint:TestPoint_Pad_2.0x2.0mm")
+    )
     (path "/2621d025-fe0d-4af8-948b-aae2ac25d436"
