File: 2-3 Pin Hardware/3-pin digital LED corner PCB.kicad_sch (KiCad schematic)
At the start: 13 parts, among them J1 Conn_01x01_Male, J10 Conn_01x01_Male, J2 Conn_01x01_Male, J3 Conn_01x01_Male, J4 Conn_01x01_Male, J5 Conn_01x01_Male, J6 Conn_01x01_Male, J7 Conn_01x01_Male, J8 Conn_01x01_Male, J9 Conn_01x01_Male

Commit message: update 2-3 pin corner PCB
Parts:
- added JP2: (no value), symbol Jumper:Jumper_3_Open
- added JP3: Jumper_3_Open, Jumper:SolderJumper-3_P1.3mm_Open_Pad1.0x1.5mm, symbol Jumper:Jumper_3_Open
Connections:
- net DOUT: now reaches D1.2 (DOUT), JP1.2 (B)
- net DOUT: now also JP2.3 (B), JP3.3 (B); no longer J5.1 (Pin_1)
- net DIN: now reaches D1.4 (DIN), JP1.1 (A)
- net DIN: now also JP2.1 (A), JP3.1 (A); no longer J2.1 (Pin_1)
- new net K1: J2.1 (Pin_1), JP2.2 (C)
- new net K2: J5.1 (Pin_1), JP3.2 (C)
Other:
- moved on the sheet: C1, J1, J2, J3, J4, J5, J6
